File: PWB.003.kicad_sch (KiCad schematic)
At the start: 48 parts, among them J1 USB_C_Receptacle_PowerOnly_6P, J2 XT30PW-F, J3 XT30PW-M, J4 BAT, J5 Conn_01x04_Pin, J6 Conn_01x05_Pin, Q1 IRLML6402TR, Q2 IRLML6402TR, Q3 2N7002, Q4 IRLML6402TR, U1 TPS63070RNMR, U2 BQ24073RGT

Commit message: Improved PCB
- Added 10k resistor on control inputs TPS63070
- Changed layout of inductor and filtering capacitors
- added legend on bottom layer
- updated DRC
- validated design on JLCDFM
Parts:
- added R13: 10k, Resistor_SMD:R_0805_2012Metric, symbol Device:R
- renumbered C3 to C10, C4 to C2, C5 to C3, C6 to C4, C7 to C5, C8 to C6, C9 to C7, C10 to C8, C2 to C9, R13 to R14, R14 to R15, R15 to R16, R16 to R17, R17 to R18, R18 to R19, R19 to R20
Connections:
- net VOUT: now also R17.1
- net VSYS: now also R13.2; no longer Q2.3 (S), R17.1, U1.1 (PS/SYNC)
- new net: Q2.3 (S), R13.1, U1.1 (PS/SYNC)
Other:
- moved on the sheet: C11, C2, C3, C4, C5, C6, C7, C8, L1, Q2, R14, R17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
